File: Pager.kicad_sch (KiCad schematic)
At the start: 18 parts, among them U1 ESP32-S3-MINI-1, Y1 ABS25-32.768KHZ-6-T

Commit message: brh
Parts:
- added F1: Fuse_Small, symbol Device:Fuse_Small
- added J2: Conn_01x02_Pin, symbol Connector:Conn_01x02_Pin
Connections:
- net Power/USBD-: now reaches U1.23 (USB_D-)
- net Power/USBD+: now reaches U1.24 (USB_D+)
- net Batt_Sense+: now reaches U1.6 (IO2)
- net Charging: now reaches U1.7 (IO3)
- new net Battery+: F1.2
- new net Battery-: J2.2 (Pin_2)
- new net V_{BATT}: F1.1, J2.1 (Pin_1)
Other:
- added sheet Buttons (buttons.kicad_sch)
- added sheet Buzzer (buzzer.kicad_sch)
- added sheet Radio (radio.kicad_sch)
- added sheet Screen (screen.kicad_sch)
- sheet Power ports: added Batt_Sense+, Charging, USBD+, USBD-; removed none
- note added: "Battery Connector"
