File: Pager/Pager.kicad_sch (KiCad schematic)
At the start: 20 parts, among them J2 Conn_01x02_Pin, U1 ESP32-S3-MINI-1, Y1 ABS25-32.768KHZ-6-T

Commit message: finished radio module
Connections:
- net RF_CSn: now reaches U1.14 (IO10)
- net RF_SI: now reaches U1.15 (IO11)
- net RF_SCLK: now reaches U1.16 (IO12)
- net RF_SO: now reaches U1.17 (IO13)
Other:
- sheet Radio ports: added RF_CSn, RF_GDO0, RF_GDO1, RF_GDO2, RF_SCLK, RF_SI; removed none
Changed lines of the file:
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@@
 	(wire
 		(pts
+			(xy 113.03 86.36) (xy 115.57 86.36)
+		)
+		(stroke
+			(width 0)
+			(type default)
+		)
+	)
+	(wire
+		(pts
 			(xy 113.03 30.48) (xy 113.03 31.75)
 		)
@@
 	(wire
 		(pts
+			(xy 113.03 91.44) (xy 115.57 91.44)
+		)
+		(stroke
+			(width 0)
+			(type default)
+		)
+	)
+	(wire
+		(pts
+			(xy 213.36 146.05) (xy 215.9 146.05)
+		)
+		(stroke
+			(width 0)
+			(type default)
+		)
+	)
+	(wire
+		(pts
 			(xy 125.73 30.48) (xy 130.81 30.48)
 		)
@@
 	(wire
 		(pts
+			(xy 113.03 88.9) (xy 115.57 88.9)
+		)
+		(stroke
+			(width 0)
+			(type default)
+		)
+	)
+	(wire
+		(pts
 			(xy 100.33 63.5) (xy 115.57 63.5)
 		)
@@
 	(wire
 		(pts
+			(xy 213.36 138.43) (xy 215.9 138.43)
+		)
+		(stroke
+			(width 0)
+			(type default)
+		)
+	)
+	(wire
+		(pts
 			(xy 93.98 39.37) (xy 93.98 40.64)
 		)
@@
 	(wire
 		(pts
+			(xy 213.36 133.35) (xy 215.9 133.35)
+		)
+		(stroke
+			(width 0)
+			(type default)
+		)
+	)
+	(wire
+		(pts
 			(xy 100.33 30.48) (xy 100.33 31.75)
 		)
@@
 	(wire
 		(pts
+			(xy 113.03 83.82) (xy 115.57 83.82)
+		)
+		(stroke
+			(width 0)
+			(type default)
+		)
+	)
+	(wire
+		(pts
 			(xy 36.83 180.34) (xy 43.18 180.34)
 		)
@@
 	(wire
 		(pts
+			(xy 213.36 140.97) (xy 215.9 140.97)
+		)
+		(stroke
+			(width 0)
+			(type default)
+		)
+	)
+	(wire
+		(pts
 			(xy 130.81 30.48) (xy 130.81 48.26)
 		)
@@
 	(wire
 		(pts
+			(xy 213.36 135.89) (xy 215.9 135.89)
+		)
+		(stroke
+			(width 0)
+			(type default)
+		)
+	)
+	(wire
+		(pts
 			(xy 255.27 62.23) (xy 256.54 62.23)
 		)
@@
 	(wire
 		(pts
+			(xy 213.36 143.51) (xy 215.9 143.51)
+		)
+		(stroke
+			(width 0)
+			(type default)
+		)
+	)
+	(wire
+		(pts
 			(xy 119.38 30.48) (xy 125.73 30.48)
 		)
@@
 		)
 	)
+	(label "RF_GDO2"
+		(at 213.36 140.97 180)
+		(effects
+			(font
+				(size 1.27 1.27)
+			)
+			(justify right bottom)
+		)
+	)
+	(label "RF_SI"
+		(at 113.03 86.36 180)
+		(effects
+			(font
+				(size 1.27 1.27)
+			)
+			(justify right bottom)
+		)
+	)
 	(label "Battery-"
 		(at 63.5 182.88 180)
@@
 		)
 	)
+	(label "RF_SCLK"
+		(at 213.36 143.51 180)
+		(effects
+			(font
+				(size 1.27 1.27)
+			)
+			(justify right bottom)
+		)
+	)
 	(label "Batt_Sense+"
 		(at 100.33 63.5 0)
@@
 		)
 	)
+	(label "RF_SO"
+		(at 113.03 91.44 180)
+		(effects
+			(font
+				(size 1.27 1.27)
+			)
+			(justify right bottom)
+		)
+	)
+	(label "RF_CSn"
+		(at 113.03 83.82 180)
+		(effects
+			(font
+				(size 1.27 1.27)
+			)
+			(justify right bottom)
+		)
+	)
+	(label "RF_SCLK"
+		(at 113.03 88.9 180)
+		(effects
+			(font
+				(size 1.27 1.27)
+			)
+			(justify right bottom)
+		)
+	)
 	(label "Battery+"
 		(at 63.5 180.34 180)
@@
 		)
 	)
+	(label "RF_SO"
+		(at 213.36 138.43 180)
+		(effects
+			(font
+				(size 1.27 1.27)
+			)
+			(justify right bottom)
+		)
+	)
+	(label "RF_CSn"
+		(at 213.36 133.35 180)
+		(effects
+			(font
+				(size 1.27 1.27)
+			)
+			(justify right bottom)
+		)
+	)
+	(label "RF_GDO0"
+		(at 213.36 135.89 180)
+		(effects
+			(font
+				(size 1.27 1.27)
+			)
+			(justify right bottom)
+		)
+	)
 	(label "Charging"
 		(at 203.2 22.86 0)
@@
 		)
 	)
+	(label "RF_SI"
+		(at 213.36 146.05 180)
+		(effects
+			(font
+				(size 1.27 1.27)
+			)
+			(justify right bottom)
+		)
+	)
 	(label "Batt_Sense+"
 		(at 203.2 20.32 0)
@@
 			)
 		)
+		(pin "RF_CSn" input
+			(at 215.9 133.35 180)
+			(effects
+				(font
+					(size 1.27 1.27)
+				)
+				(justify left)
+			)
+		)
+		(pin "RF_GDO0" input
+			(at 215.9 135.89 180)
+			(effects
+				(font
+					(size 1.27 1.27)
+				)
+				(justify left)
+			)
+		)
+		(pin "RF_GDO1" input
+			(at 215.9 138.43 180)
+			(effects
+				(font
+					(size 1.27 1.27)
+				)
+				(justify left)
+			)
+		)
+		(pin "RF_GDO2" input
+			(at 215.9 140.97 180)
+			(effects
+				(font
+					(size 1.27 1.27)
+				)
+				(justify left)
+			)
+		)
+		(pin "RF_SCLK" input
+			(at 215.9 143.51 180)
+			(effects
+				(font
+					(size 1.27 1.27)
+				)
+				(justify left)
+			)
+		)
+		(pin "RF_SI" input
+			(at 215.9 146.05 180)
+			(effects
+				(font
+					(size 1.27 1.27)
+				)
+				(justify left)
+			)
+		)

Commit message: br
Connections:
- net Buttons/Button_3: now reaches U1.10 (IO6)
- net Buttons/Button_4: now reaches U1.11 (IO7)
- net Buttons/Button_5: now reaches U1.12 (IO8)
- net Buttons/Button_1: now reaches U1.8 (IO4)
- net Buttons/Button_2: now reaches U1.9 (IO5)
- net RF_CSn: no longer names the net of U1.14 (IO10)
- net RF_SCLK: no longer names the net of U1.16 (IO12)
- net RF_SI: no longer names the net of U1.15 (IO11)
- net RF_SO: no longer names the net of U1.17 (IO13)
Other:
- sheet Buttons ports: added Button_1, Button_2, Button_3, Button_4, Button_5; removed none
- sheet Radio ports: added none; removed RF_CSn, RF_GDO0, RF_GDO1, RF_GDO2, RF_SCLK, RF_SI
