File: Pager/buttons.kicad_sch (KiCad schematic)
At the start: 0 parts

Commit message: br
Parts:
- added C14, C15, C16, C17, C18: 100nF, Package_SO:SOIC-8_3.9x4.9mm_P1.27mm, symbol Device:C_Small
- added R10, R12, R14, R16, R18: 1k, symbol Device:R_Small
- added R11, R13, R15, R17, R9: 10k, symbol Device:R_Small
- added SW2, SW3, SW4, SW5, SW6: SW_Push, Button_Switch_SMD:Nidec_Copal_CAS-120A, symbol Switch:SW_Push
Connections:
- new net: R17.2, R18.1, SW6.1
- new net: R10.1, R9.2, SW2.1
- new net: R11.2, R12.1, SW3.1
- new net: R13.2, R14.1, SW4.1
- new net: R15.2, R16.1, SW5.1
- new net +3V3: R11.1, R13.1, R15.1, R17.1, R9.1
- new net Button_1: C14.1, R10.2
- new net Button_2: C15.1, R12.2
- new net Button_3: C16.1, R14.2
- new net Button_4: C17.1, R16.2
- new net Button_5: C18.1, R18.2
- new net GND: C14.2, C15.2, C16.2, C17.2, C18.2, SW2.2, SW3.2, SW4.2, SW5.2, SW6.2

Commit message: Schematic Review, Footprints Added, Need Screen
Parts:
- C29: renamed from C14; footprint Package_SO:SOIC-8_3.9x4.9mm_P1.27mm -> Capacitor_SMD:C_0603_1608Metric
- C30: renamed from C15; footprint Package_SO:SOIC-8_3.9x4.9mm_P1.27mm -> Capacitor_SMD:C_0603_1608Metric
- C31: renamed from C16; footprint Package_SO:SOIC-8_3.9x4.9mm_P1.27mm -> Capacitor_SMD:C_0603_1608Metric
- C32: renamed from C17; footprint Package_SO:SOIC-8_3.9x4.9mm_P1.27mm -> Capacitor_SMD:C_0603_1608Metric
- C33: renamed from C18; footprint Package_SO:SOIC-8_3.9x4.9mm_P1.27mm -> Capacitor_SMD:C_0603_1608Metric
- R16: renamed from R9; footprint (none) -> Resistor_SMD:R_0603_1608Metric
- R17: renamed from R11; footprint (none) -> Resistor_SMD:R_0603_1608Metric
- R18: renamed from R13; footprint (none) -> Resistor_SMD:R_0603_1608Metric
- R19: renamed from R10; footprint (none) -> Resistor_SMD:R_0603_1608Metric
- R20: renamed from R12; footprint (none) -> Resistor_SMD:R_0603_1608Metric
- R21: renamed from R14; footprint (none) -> Resistor_SMD:R_0603_1608Metric
- R22: renamed from R15; footprint (none) -> Resistor_SMD:R_0603_1608Metric
- R23: renamed from R17; footprint (none) -> Resistor_SMD:R_0603_1608Metric
- R24: renamed from R16; footprint (none) -> Resistor_SMD:R_0603_1608Metric
- R25: renamed from R18; footprint (none) -> Resistor_SMD:R_0603_1608Metric
- SW2, SW3, SW4, SW5, SW6: footprint Button_Switch_SMD:Nidec_Copal_CAS-120A -> Button_Switch_THT:SW_PUSH_6mm

Commit message: layout
Parts:
- C29, C30, C31, C32, C33: footprint Capacitor_SMD:C_0603_1608Metric -> Capacitor_SMD:C_0805_2012Metric_Pad1.18x1.45mm_HandSolder
- R16, R17, R18, R19, R20, R21, R22, R23, R24, R25: footprint Resistor_SMD:R_0603_1608Metric -> Resistor_SMD:R_0805_2012Metric_Pad1.20x1.40mm_HandSolder
Changed lines of the file:
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@@
 			)
 		)
-		(property "Footprint" "Resistor_SMD:R_0603_1608Metric"
+		(property "Footprint" "Resistor_SMD:R_0805_2012Metric_Pad1.20x1.40mm_HandSolder"
 			(at 88.9 74.93 0)
 			(hide yes)
@@
 			)
 		)
-		(property "Footprint" "Resistor_SMD:R_0603_1608Metric"
+		(property "Footprint" "Resistor_SMD:R_0805_2012Metric_Pad1.20x1.40mm_HandSolder"
 			(at 35.56 31.75 0)
 			(hide yes)
@@
 			)
 		)
-		(property "Footprint" "Resistor_SMD:R_0603_1608Metric"
+		(property "Footprint" "Resistor_SMD:R_0805_2012Metric_Pad1.20x1.40mm_HandSolder"
 			(at 48.26 102.87 0)
 			(hide yes)
@@
 			)
 		)
-		(property "Footprint" "Resistor_SMD:R_0603_1608Metric"
+		(property "Footprint" "Resistor_SMD:R_0805_2012Metric_Pad1.20x1.40mm_HandSolder"
 			(at 48.26 71.12 0)
 			(hide yes)
@@
 			)
 		)
-		(property "Footprint" "Resistor_SMD:R_0603_1608Metric"
+		(property "Footprint" "Resistor_SMD:R_0805_2012Metric_Pad1.20x1.40mm_HandSolder"
 			(at 46.99 35.56 0)
 			(hide yes)
@@
 			)
 		)
-		(property "Footprint" "Resistor_SMD:R_0603_1608Metric"
+		(property "Footprint" "Resistor_SMD:R_0805_2012Metric_Pad1.20x1.40mm_HandSolder"
 			(at 36.83 67.31 0)
 			(hide yes)
@@
 			)
 		)
-		(property "Footprint" "Resistor_SMD:R_0603_1608Metric"
+		(property "Footprint" "Resistor_SMD:R_0805_2012Metric_Pad1.20x1.40mm_HandSolder"
 			(at 97.79 36.83 0)
 			(hide yes)
@@
 			)
 		)
-		(property "Footprint" "Resistor_SMD:R_0603_1608Metric"
+		(property "Footprint" "Resistor_SMD:R_0805_2012Metric_Pad1.20x1.40mm_HandSolder"
 			(at 36.83 99.06 0)
 			(hide yes)
@@
 			)
 		)
-		(property "Footprint" "Capacitor_SMD:C_0603_1608Metric"
+		(property "Footprint" "Capacitor_SMD:C_0805_2012Metric_Pad1.18x1.45mm_HandSolder"
 			(at 53.34 109.22 0)
 			(hide yes)
@@
 			)
 		)
-		(property "Footprint" "Capacitor_SMD:C_0603_1608Metric"
+		(property "Footprint" "Capacitor_SMD:C_0805_2012Metric_Pad1.18x1.45mm_HandSolder"
 			(at 52.07 41.91 0)
 			(hide yes)
@@
 			)
 		)
-		(property "Footprint" "Capacitor_SMD:C_0603_1608Metric"
+		(property "Footprint" "Capacitor_SMD:C_0805_2012Metric_Pad1.18x1.45mm_HandSolder"
 			(at 105.41 85.09 0)
 			(hide yes)
@@
 			)
 		)
-		(property "Footprint" "Capacitor_SMD:C_0603_1608Metric"
+		(property "Footprint" "Capacitor_SMD:C_0805_2012Metric_Pad1.18x1.45mm_HandSolder"
 			(at 102.87 43.18 0)
 			(hide yes)
@@
 			)
 		)
-		(property "Footprint" "Resistor_SMD:R_0603_1608Metric"
+		(property "Footprint" "Resistor_SMD:R_0805_2012Metric_Pad1.20x1.40mm_HandSolder"
 			(at 100.33 78.74 0)
 			(hide yes)
@@
 			)
 		)
-		(property "Footprint" "Resistor_SMD:R_0603_1608Metric"
+		(property "Footprint" "Resistor_SMD:R_0805_2012Metric_Pad1.20x1.40mm_HandSolder"
 			(at 86.36 33.02 0)
 			(hide yes)
@@
 			)
 		)
-		(property "Footprint" "Capacitor_SMD:C_0603_1608Metric"
+		(property "Footprint" "Capacitor_SMD:C_0805_2012Metric_Pad1.18x1.45mm_HandSolder"
 			(at 53.34 77.47 0)
 			(hide yes)
