File: Pager/radio.kicad_sch (KiCad schematic)
At the start: 0 parts

Commit message: created new radio symbol and started on radio schem
Parts:
- added C10, C11, C12, C13, C9: C_Small, symbol Device:C_Small
- added C4: 100 nF, symbol Device:C_Small
- added C7, C8: 27 pF ± 5%, symbol Device:C_Small
- added L1, L2, L3, L4, L5, L6: L_Small, symbol Device:L_Small
- added R5: R_Small, symbol Device:R_Small
- added U5: CC1101RGPR, symbol Custom_Pager_Symbol_Library:CC1101RGPR
- added Y2: 26 MHz, symbol Device:Crystal_Small
Connections:
- new net: C7.1, U5.8 (XOSC_Q1), Y2.1
- new net: C8.1, U5.10 (XOSC_Q2), Y2.2
- new net: C9.1, L3.1
- new net: C10.1, C12.1, L1.1, L4.2
- new net: C10.2, C11.1, L2.1, L3.2
- new net: L2.2, U5.12 (RF_P)
- new net: C11.2, L4.1, L5.2
- new net: C13.2, L5.1, L6.2
- new net: R5.1, U5.17 (RBIAS)
- new net: C4.1, U5.5 (DCOUPL)
- new net: L1.2, U5.13 (RF_N)
- new net GND: C12.2, C13.1, C4.2, C7.2, C8.2, C9.2, R5.2, U5.16 (GND), U5.19 (GND), U5.21 (EP_GND)
Other:
- note added: "Pin for exposed die ground"

Commit message: add cap values
Parts:
- C10: value C_Small -> 1.0 pF
- C11, C12: value C_Small -> 1.5 pF
- C13: value C_Small -> 3.3 pF
- C7, C8: value 27 pF ± 5% -> 27 pF
- C9: value C_Small -> 100 pF
Changed lines of the file:
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@@
 			)
 		)
-		(property "Value" "C_Small"
+		(property "Value" "100 pF"
 			(at 132.08 110.4899 0)
 			(show_name no)
@@
 		(in_pos_files yes)
 		(dnp no)
-		(fields_autoplaced yes)
 		(property "Reference" "C10"
 			(at 127 92.7099 0)
@@
 			)
 		)
-		(property "Value" "C_Small"
-			(at 127 95.2499 0)
+		(property "Value" "1.0 pF"
+			(at 127 94.996 0)
 			(show_name no)
 			(do_not_autoplace no)
@@
 			)
 		)
-		(property "Value" "27 pF ± 5%"
+		(property "Value" "27 pF"
 			(at 100.33 124.4599 0)
 			(show_name no)
@@
 			)
 		)
-		(property "Value" "C_Small"
+		(property "Value" "1.5 pF"
 			(at 130.81 82.5499 0)
 			(show_name no)
@@
 			(effects
 				(font
+					(face "KiCad Font")
 					(size 1.27 1.27)
 				)
@@
 		(in_pos_files yes)
 		(dnp no)
-		(fields_autoplaced yes)
 		(property "Reference" "C11"
 			(at 139.7 92.71 90)
@@
 			)
 		)
-		(property "Value" "C_Small"
-			(at 139.7 95.25 90)
+		(property "Value" "1.5 pF"
+			(at 139.7 95.504 90)
 			(show_name no)
 			(do_not_autoplace no)
@@
 			)
 		)
-		(property "Value" "27 pF ± 5%"
+		(property "Value" "27 pF"
 			(at 87.63 124.4599 0)
 			(show_name no)
@@
 			)
 		)
-		(property "Value" "C_Small"
+		(property "Value" "3.3 pF"
 			(at 154.94 99.0599 0)
 			(show_name no)

Commit message: finish radio ic
Parts:
- added AE1: Antenna, Package_DFN_QFN:DFN-8-1EP_2x3mm_P0.5mm_EP0.61x2.2mm, symbol Device:Antenna
- added C14: 12 pF, symbol Device:C_Small
- added C15: 47 pF, symbol Device:C_Small
- added C17, C18, C20, C21: 100nF, symbol Device:C_Small
- added L7: 3.3 nH, Relay_THT:Relay_DPDT_Finder_30.22, symbol Device:L_Small
- L1, L2, L5, L6: value L_Small -> 12 nH
- L3, L4: value L_Small -> 18 nH
- R5: value R_Small -> 56 kΩ
Connections:
- net GND: now also C17.2, C18.1, C20.2, C21.2
- net at L6.1: now also C14.1, C15.2
- net RF_SCLK: now reaches U5.1 (SCLK)
- net +3.3V: now reaches U5.11 (AVDD)
- net +3.3V: now also U5.14 (AVDD), U5.15 (AVDD), U5.18 (DGUARD), U5.4 (DVDD), U5.9 (AVDD), C17.1, C18.2, C20.1, C21.1
- net RF_GDO1: now reaches U5.2 (SO_(GDO1))
- net RF_SI: now reaches U5.20 (SI)
- net RF_GDO2: now reaches U5.3 (GDO2)
- net RF_GDO0: now reaches U5.6 (GDO0)
- net RF_CSn: now reaches U5.7 (CSn)
- new net: C15.1, L7.1
- new net: AE1.1 (A), C14.2, L7.2
Other:
- moved on the sheet: C10, C11, C12, C13, C7, C8, C9, L1, L2, L3, L4, L5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

Commit message: finished radio module
Changed lines of the file:
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@@
 		)
 	)
-	(label "RF_GDO1"
+	(hierarchical_label "RF_GDO0"
+		(shape input)
+		(at 54.61 114.3 180)
+		(effects
+			(font
+				(size 1.27 1.27)
+			)
+			(justify right)
+		)
+	)
+	(hierarchical_label "RF_GDO2"
+		(shape input)
+		(at 58.42 92.71 180)
+		(effects
+			(font
+				(size 1.27 1.27)
+			)
+			(justify right)
+		)
+	)
+	(hierarchical_label "RF_GDO1"
+		(shape input)
 		(at 58.42 88.9 180)
 		(effects
@@
 				(size 1.27 1.27)
 			)
-			(justify right bottom)
+			(justify right)
 		)
 	)
-	(label "RF_GDO0"
-		(at 54.61 114.3 180)
+	(hierarchical_label "RF_CSn"
+		(shape input)
+		(at 54.61 119.38 180)
 		(effects
 			(font
 				(size 1.27 1.27)
 			)
-			(justify right bottom)
+			(justify right)
 		)
 	)
-	(label "RF_GDO2"
-		(at 58.42 92.71 180)
-		(effects
-			(font
-				(size 1.27 1.27)
-			)
-			(justify right bottom)
-		)
-	)
-	(label "RF_SI"
+	(hierarchical_label "RF_SI"
+		(shape input)
 		(at 58.42 67.31 180)
 		(effects
@@
 				(size 1.27 1.27)
 			)
-			(justify right bottom)
+			(justify right)
 		)
 	)
-	(label "RF_CSn"
-		(at 54.61 119.38 180)
-		(effects
-			(font
-				(size 1.27 1.27)
-			)
-			(justify right bottom)
-		)
-	)
-	(label "RF_SCLK"
+	(hierarchical_label "RF_SCLK"
+		(shape input)
 		(at 58.42 85.09 180)
 		(effects
@@
 				(size 1.27 1.27)
 			)
-			(justify right bottom)
+			(justify right)
 		)
 	)

Commit message: Schematic Review, Footprints Added, Need Screen
Parts:
- removed C15: 47 pF, symbol Device:C_Small
- removed L7: 3.3 nH, Relay_THT:Relay_DPDT_Finder_30.22, symbol Device:L_Small
- removed Y2: 26 MHz, symbol Device:Crystal_Small
- added C10, C9: C_Small, Capacitor_SMD:C_0402_1005Metric, symbol Device:C_Small
- added R28: 0, Resistor_SMD:R_0402_1005Metric, symbol Device:R_Small
- added Y1: 26 MHz, Crystal:Crystal_SMD_3225-4Pin_3.2x2.5mm, symbol Device:Crystal_GND24_Small
- AE1: footprint Package_DFN_QFN:DFN-8-1EP_2x3mm_P0.5mm_EP0.61x2.2mm -> Antenna:ANT_0915AT43A0026E_JOT
- C15: renamed from C21; footprint (none) -> Capacitor_SMD:C_0402_1005Metric
- C16: renamed from C4; footprint (none) -> Capacitor_SMD:C_0402_1005Metric
- C17: renamed from C7; value 27 pF -> 15 pF; footprint (none) -> Capacitor_SMD:C_0402_1005Metric
- C18: renamed from C20; footprint (none) -> Capacitor_SMD:C_0402_1005Metric
- C19: renamed from C8; value 27 pF -> 15 pF; footprint (none) -> Capacitor_SMD:C_0402_1005Metric
- C20: renamed from C18; footprint (none) -> Capacitor_SMD:C_0402_1005Metric
- C21: renamed from C17; footprint (none) -> Capacitor_SMD:C_0402_1005Metric
- C22: renamed from C10; footprint (none) -> Capacitor_SMD:C_0402_1005Metric
- C23: renamed from C9; footprint (none) -> Capacitor_SMD:C_0402_1005Metric
- C24: renamed from C12; footprint (none) -> Capacitor_SMD:C_0402_1005Metric
- C25: renamed from C11; footprint (none) -> Capacitor_SMD:C_0402_1005Metric
- C26: renamed from C13; footprint (none) -> Capacitor_SMD:C_0402_1005Metric
- C28: renamed from C14; value 12 pF -> 100pF; footprint (none) -> Capacitor_SMD:C_0402_1005Metric
- L1, L2, L3, L4, L5, L6: footprint (none) -> Inductor_SMD:L_0402_1005Metric
- R13: renamed from R5; footprint (none) -> Resistor_SMD:R_0402_1005Metric
- U4: renamed from U5; footprint (none) -> Package_DFN_QFN:Texas_RGP0020H_VQFN-20-1EP_4x4mm_P0.5mm_EP2.4x2.4mm_ThermalVias
Connections:
- net GND: now also C10.2, C9.2, Y1.2 (G), Y1.4 (G)
- net at C17.1, U4.8 (XOSC_Q1): now also Y1.1
- net at C19.1, U4.10 (XOSC_Q2): now also Y1.3
- net at C28.2: now also C9.1, R28.1; no longer AE1.1 (A)
- net +3.3V renamed +3V3
- new net: AE1.1 (A), C10.1, R28.2
Other:
- moved on the sheet: AE1

Commit message: updated
Parts:
- removed C28: 100pF, Capacitor_SMD:C_0402_1005Metric, symbol Device:C_Small
- removed R28: 0, Resistor_SMD:R_0402_1005Metric, symbol Device:R_Small
- added L7: 3.3nH, symbol Device:L_Small
- C10: value C_Small -> 12pF; footprint Capacitor_SMD:C_0402_1005Metric -> (none); now fitted
- C15, C16, C17, C18, C19, C20, C21, C22, C23, C24, C25, C26: footprint Capacitor_SMD:C_0402_1005Metric -> Capacitor_SMD:C_0805_2012Metric_Pad1.18x1.45mm_HandSolder
- C9: value C_Small -> 47pF; footprint Capacitor_SMD:C_0402_1005Metric -> (none); now fitted
- L1, L2, L3, L4, L5, L6: footprint Inductor_SMD:L_0402_1005Metric -> Inductor_SMD:L_0805_2012Metric_Pad1.05x1.20mm_HandSolder
Connections:
- net GND: no longer C10.2, C9.2
- net at L6.1: now also C10.1, C9.1
- net at AE1.1 (A): now also C10.2, L7.2; no longer C10.1
- new net: C9.2, L7.1

Commit message: layout
Parts:
- C10, C9: footprint (none) -> Capacitor_SMD:C_0805_2012Metric_Pad1.18x1.45mm_HandSolder
- L7: footprint (none) -> Inductor_SMD:L_0805_2012Metric_Pad1.05x1.20mm_HandSolder
- R13: footprint Resistor_SMD:R_0402_1005Metric -> Resistor_SMD:R_0805_2012Metric_Pad1.20x1.40mm_HandSolder
Changed lines of the file:
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@@
 			)
 		)
-		(property "Footprint" ""
+		(property "Footprint" "Inductor_SMD:L_0805_2012Metric_Pad1.05x1.20mm_HandSolder"
 			(at 207.01 102.87 0)
 			(hide yes)
@@
 			)
 		)
-		(property "Footprint" ""
+		(property "Footprint" "Capacitor_SMD:C_0805_2012Metric_Pad1.18x1.45mm_HandSolder"
 			(at 196.85 92.71 0)
 			(hide yes)
@@
 			)
 		)
-		(property "Footprint" ""
+		(property "Footprint" "Capacitor_SMD:C_0805_2012Metric_Pad1.18x1.45mm_HandSolder"
 			(at 198.12 102.87 0)
 			(hide yes)
@@
 			)
 		)
-		(property "Footprint" "Resistor_SMD:R_0402_1005Metric"
+		(property "Footprint" "Resistor_SMD:R_0805_2012Metric_Pad1.20x1.40mm_HandSolder"
 			(at 96.52 60.96 0)
 			(hide yes)
