File: Pager/Pager.kicad_pcb (KiCad board)
At the start: 2 copper layers, 98 parts, among them J1 Conn_01x02_Pin, J3 USB4085-GF-A_REVB, Q1 AO3400A, Q2 AO3401A, SW1 SW_SPDT, SW2 SW_Push, SW3 SW_Push, SW4 SW_Push, SW5 SW_Push, SW6 SW_Push, U1 ESP32-S3-MINI-1, U2 AP2112K-3.3, U3 MCP73831-2-OT, U4 CC1101RGPR, U5 USBLC6-2SC6, Y1 26 MHz

Commit message: layout
Parts:
- removed the C9 at (80.1, 82.5)
- moved C10 168.3 mm to (244.9, 50.8)
- moved C15 168.3 mm to (244.9, 52.8)
- moved C16 168.3 mm to (244.9, 54.8)
- moved C18 168.3 mm to (244.9, 58.7)
- moved C19 168.3 mm to (247.8, 48.9)
- moved C20 168.3 mm to (247.8, 50.8)
- moved C21 168.3 mm to (247.8, 52.8)
- moved C23 168.3 mm to (247.8, 56.7)
- moved C24 168.3 mm to (247.8, 58.7)
- moved C25 168.3 mm to (250.7, 48.9)
- moved L3 168.3 mm to (242.1, 52.8)
- moved L6 168.3 mm to (242.1, 58.8)
- moved Y1 168.3 mm to (252.8, 62.0)
- moved R9 166.7 mm to (220.9, 69.0), turned to 90 degrees
- moved R5 156.6 mm to (205.2, 69.1)
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
Commit message: esp32
Parts:
- moved C28 141.8 mm to (226.5, 104.4)
- moved D1 141.8 mm to (209.6, 107.5)
- moved D2 141.8 mm to (248.2, 99.1)
- moved Q1 141.8 mm to (243.5, 94.8)
- moved R10 141.8 mm to (196.0, 110.6)
- moved R14 141.8 mm to (248.0, 93.9)
- moved R15 141.8 mm to (248.0, 96.4)
- moved R26 141.8 mm to (243.3, 98.5)
- moved R8 141.8 mm to (196.0, 101.7)
- moved TP1 141.8 mm to (190.4, 85.9)
- moved TP2 141.8 mm to (190.4, 89.5)
- moved TP5 141.8 mm to (197.5, 85.9)
- moved TP6 141.8 mm to (197.5, 89.5)
- moved U3 141.8 mm to (205.0, 106.5)
- moved C12 141.8 mm to (200.4, 105.8)
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Routing:
- added copper zone on B.Cu, net GND
Other:
- board outline added: 65.2 x 35.6 mm
