File: Pager/Display.kicad_sch (KiCad schematic)
At the start: 0 parts

Commit message: add display module
Parts:
- added J2: Conn_01x04, Package_DIP:DIP-20_W7.62mm, symbol Connector_Generic:Conn_01x04
Connections:
- new net +3V3: J2.3 (Pin_3)
- new net GND: J2.4 (Pin_4)
- new net SCK: J2.2 (Pin_2)
- new net SDA: J2.1 (Pin_1)
